Commit message: Added TF prefix and files for costmap.

File: turtlebot3_description/urdf/turtlebot3_senseless_waffle.gazebo.xacro (robot description, xacro)
@@ -2,4 +2,6 @@
 <robot name="turtlebot3_senseless_waffle_sim" xmlns:xacro="http://ros.org/wiki/xacro">
   <xacro:arg name="imu_visual"    default="false"/>
+  <xacro:arg name="mu_value"      default="20"/>
+  <xacro:arg name="tf_prefix"     default=""/>
   <gazebo reference="base_link">
     <material>Gazebo/DarkGrey</material>
@@ -9,6 +11,6 @@
   </gazebo>
   <gazebo reference="wheel_left_link">
-    <mu1>0.1</mu1>
-    <mu2>0.1</mu2>
+    <mu1>$(arg mu_value)</mu1>
+    <mu2>$(arg mu_value)</mu2>
     <kp>500000.0</kp>
     <kd>10.0</kd>
@@ -19,6 +21,6 @@
   </gazebo>
   <gazebo reference="wheel_right_link">
-    <mu1>0.1</mu1>
-    <mu2>0.1</mu2>
+    <mu1>$(arg mu_value)</mu1>
+    <mu2>$(arg mu_value)</mu2>
     <kp>500000.0</kp>
     <kd>10.0</kd>
@@ -29,6 +31,6 @@
   </gazebo>
   <gazebo reference="caster_back_right_link">
-    <mu1>0.1</mu1>
-    <mu2>0.1</mu2>
+    <mu1>$(arg mu_value)</mu1>
+    <mu2>$(arg mu_value)</mu2>
     <kp>1000000.0</kp>
     <kd>100.0</kd>
@@ -38,6 +40,6 @@
   </gazebo>
   <gazebo reference="caster_back_left_link">
-    <mu1>0.1</mu1>
-    <mu2>0.1</mu2>
+    <mu1>$(arg mu_value)</mu1>
+    <mu2>$(arg mu_value)</mu2>
     <kp>1000000.0</kp>
     <kd>100.0</kd>
@@ -57,8 +59,8 @@
       <commandTopic>cmd_vel</commandTopic>
       <odometryTopic>odom</odometryTopic>
-      <odometryFrame>odom</odometryFrame>
+      <odometryFrame>$(arg tf_prefix)/odom</odometryFrame>
       <odometrySource>world</odometrySource>
       <publishOdomTF>true</publishOdomTF>
-      <robotBaseFrame>base_footprint</robotBaseFrame>
+      <robotBaseFrame>$(arg tf_prefix)/base_footprint</robotBaseFrame>
       <publishWheelTF>false</publishWheelTF>
       <publishTf>true</publishTf>

File: turtlebot3_description/urdf/turtlebot3_senseless_waffle.urdf.xacro (robot description, xacro)
@@ -3,7 +3,8 @@
   <xacro:include filename="$(find turtlebot3_description)/urdf/common_properties.xacro"/>
   <xacro:include filename="$(find turtlebot3_description)/urdf/turtlebot3_senseless_waffle.gazebo.xacro"/>
-  <link name="base_footprint"/>
+  <xacro:arg name="tf_prefix" default=""/>
+  <link name="$(arg tf_prefix)/base_footprint"/>
   <joint name="base_joint" type="fixed">
-    <parent link="base_footprint"/>
+    <parent link="$(arg tf_prefix)/base_footprint"/>
     <child link="base_link" />
     <origin xyz="0 0 0.010" rpy="0 0 0"/>

Commit message: Handled ROS frame errors.

File: turtlebot3_description/urdf/turtlebot3_senseless_waffle.gazebo.xacro (robot description, xacro)
@@ -4,4 +4,11 @@
   <xacro:arg name="mu_value"      default="20"/>
   <xacro:arg name="tf_prefix"     default=""/>
+  <xacro:property name="tf_prefix" value="$(arg tf_prefix)"/>
+  <xacro:property name="odom_frame" value="odom"/>
+  <xacro:property name="robot_base_frame" value="base_footprint"/>
+  <xacro:if value="${tf_prefix != ''}">
+    <xacro:property name="robot_base_frame" value="${tf_prefix}/${robot_base_frame}"/>
+    <xacro:property name="odom_frame" value="${tf_prefix}/${odom_frame}"/>
+  </xacro:if>
   <gazebo reference="base_link">
     <material>Gazebo/DarkGrey</material>
@@ -59,8 +66,8 @@
       <commandTopic>cmd_vel</commandTopic>
       <odometryTopic>odom</odometryTopic>
-      <odometryFrame>$(arg tf_prefix)/odom</odometryFrame>
+      <odometryFrame>${odom_frame}</odometryFrame>
       <odometrySource>world</odometrySource>
       <publishOdomTF>true</publishOdomTF>
-      <robotBaseFrame>$(arg tf_prefix)/base_footprint</robotBaseFrame>
+      <robotBaseFrame>${robot_base_frame}</robotBaseFrame>
       <publishWheelTF>false</publishWheelTF>
       <publishTf>true</publishTf>

File: turtlebot3_description/urdf/turtlebot3_senseless_waffle.urdf.xacro (robot description, xacro)
@@ -3,8 +3,13 @@
   <xacro:include filename="$(find turtlebot3_description)/urdf/common_properties.xacro"/>
   <xacro:include filename="$(find turtlebot3_description)/urdf/turtlebot3_senseless_waffle.gazebo.xacro"/>
-  <xacro:arg name="tf_prefix" default=""/>
-  <link name="$(arg tf_prefix)/base_footprint"/>
+  <xacro:arg name="tf_prefix"     default=""/>
+  <xacro:property name="tf_prefix" value="$(arg tf_prefix)"/>
+  <xacro:property name="base_footprint_frame" value="base_footprint"/>
+  <xacro:if value="${tf_prefix != ''}">
+    <xacro:property name="base_footprint_frame" value="${tf_prefix}/${base_footprint_frame}"/>
+  </xacro:if>
+  <link name="${base_footprint_frame}"/>
   <joint name="base_joint" type="fixed">
-    <parent link="$(arg tf_prefix)/base_footprint"/>
+    <parent link="${base_footprint_frame}"/>
     <child link="base_link" />
     <origin xyz="0 0 0.010" rpy="0 0 0"/>

Commit message: Fixed issues related to namespacing.

File: turtlebot3_description/urdf/turtlebot3_senseless_waffle.gazebo.xacro (robot description, xacro)
@@ -1,13 +1,20 @@
 <?xml version="1.0"?>
 <robot name="turtlebot3_senseless_waffle_sim" xmlns:xacro="http://ros.org/wiki/xacro">
-  <xacro:arg name="imu_visual"    default="false"/>
-  <xacro:arg name="mu_value"      default="20"/>
-  <xacro:arg name="tf_prefix"     default=""/>
+  <xacro:arg name="imu_visual"  default="false"/>
+  <xacro:arg name="mu_value"    default="20"/>
+  <xacro:arg name="tf_prefix"   default=""/>
   <xacro:property name="tf_prefix" value="$(arg tf_prefix)"/>
-  <xacro:property name="odom_frame" value="odom"/>
-  <xacro:property name="robot_base_frame" value="base_footprint"/>
+  <xacro:property name="odom_frame_base_name" value="odom"/>
+  <xacro:property name="robot_base_frame_base_name" value="base_footprint"/>
+  <xacro:property name="imu_link_frame_base_name" value="imu_link"/>
   <xacro:if value="${tf_prefix != ''}">
-    <xacro:property name="robot_base_frame" value="${tf_prefix}/${robot_base_frame}"/>
-    <xacro:property name="odom_frame" value="${tf_prefix}/${odom_frame}"/>
+    <xacro:property name="odom_frame" value="${tf_prefix}/${odom_frame_base_name}"/>
+    <xacro:property name="robot_base_frame" value="${tf_prefix}/${robot_base_frame_base_name}"/>
+    <xacro:property name="imu_body_name" value="${tf_prefix}/${imu_link_frame_base_name}"/>
+  </xacro:if>
+  <xacro:if value="${tf_prefix == ''}">
+    <xacro:property name="odom_frame" value="${odom_frame_base_name}"/>
+    <xacro:property name="robot_base_frame" value="${robot_base_frame_base_name}"/>
+    <xacro:property name="imu_body_name" value="${imu_link_frame_base_name}"/>
   </xacro:if>
   <gazebo reference="base_link">
@@ -87,6 +94,6 @@
     <plugin name="imu_plugin" filename="libgazebo_ros_imu.so">
       <alwaysOn>true</alwaysOn>
-      <bodyName>imu_link</bodyName>
-      <frameName>imu_link</frameName>
+      <bodyName>${imu_link_frame_base_name}</bodyName>
+      <frameName>${imu_body_name}</frameName>
       <topicName>imu</topicName>
       <serviceName>imu_service</serviceName>

File: turtlebot3_description/urdf/turtlebot3_senseless_waffle.urdf.xacro (robot description, xacro)
@@ -4,9 +4,12 @@
   <xacro:include filename="$(find turtlebot3_description)/urdf/turtlebot3_senseless_waffle.gazebo.xacro"/>
   <xacro:arg name="tf_prefix"     default=""/>
-  <xacro:property name="tf_prefix" value="$(arg tf_prefix)"/>
+  <!-- <xacro:property name="tf_prefix" value="$(arg tf_prefix)"/> -->
   <xacro:property name="base_footprint_frame" value="base_footprint"/>
-  <xacro:if value="${tf_prefix != ''}">
-    <xacro:property name="base_footprint_frame" value="${tf_prefix}/${base_footprint_frame}"/>
+  <!-- <xacro:if value="${tf_prefix != ''}">
+    <xacro:property name="base_footprint_frame" value="${tf_prefix}/${base_footprint_frame_base_name}"/>
   </xacro:if>
+  <xacro:if value="${tf_prefix == ''}">
+    <xacro:property name="base_footprint_frame" value="${base_footprint_frame_base_name}"/>
+  </xacro:if> -->
   <link name="${base_footprint_frame}"/>
   <joint name="base_joint" type="fixed">
